File: hardware/PCB/wifi.sch (KiCad schematic (older format))
At the start: 1 part

Commit message: update pcb,
Parts:
- removed U?: RTL8723BS, symbol taobao-components:RTL8723BS
- added AE?: Antenna_Shield, symbol Device:Antenna_Shield
- added J?: Conn_01x03, symbol Connector_Generic:Conn_01x03
- added J?: Conn_01x06, symbol Connector_Generic:Conn_01x06
- added U?: RTL8723BS, symbol taobao-components:RTL8723BS
- added U?: 10KΩ,(1002),±1%,0603,C25804, w_smd_resistors:r_0603, symbol sz_jlc_resistor:10KΩ,(1002),±1%,0603,C25804
- added U? (x5): 47KΩ,(4702),±1%,0603,C25819, w_smd_resistors:r_0603, symbol sz_jlc_resistor:47KΩ,(4702),±1%,0603,C25819
- added U? (x2): 100KΩ,(1003),±1%,0603,C25803, w_smd_resistors:r_0603, symbol sz_jlc_resistor:100KΩ,(1003),±1%,0603,C25803
- added U?: 33pF,(330),±5%,50V,C0G,0603,C1663, w_smd_cap:c_0603, symbol sz_jlc_capacitor:33pF,(330),±5%,50V,C0G,0603,C1663
Connections:
- new net: U?.1, U?.12 (WL_REG)
- new net: U?.1, U?.2 (WL_BT_ANT)
- new net: U?.2, U?.23 (VIN_LDO)
- new net: U?.2, U?.34 (BT_RST)
- new net: J?.1 (Pin_1), U?.42 (UART_TXD)
- new net: J?.2 (Pin_2), U?.43 (UART_RXD)
- new net: J?.3 (Pin_3), U?.44 (UART_CTS)
- new net: AE?.1 (A), U?.2
- new net +3V3: U?.1, U?.1, U?.2, U?.2, U?.2, U?.2, U?.2, U?.2, U?.22 (VDD_IO), U?.9 (VCC)
- new net BT_H_WK: U?.7 (BT_H_WK)
- new net BT_WK: U?.6 (BT_WK)
- new net GND: AE?.2 (Shield), U?.1 (GND1), U?.20 (GND), U?.3 (GND3), U?.31 (GND), U?.33 (GND), U?.36 (GND), U?.41 (UART_RTS)
- new net SDC1_CLK: J?.3 (Pin_3), U?.17 (SDIO_CLK)
- new net SDC1_CMD: J?.4 (Pin_4), U?.1, U?.16 (SDIO_CMD)
- new net SDC1_D0: J?.2 (Pin_2), U?.1, U?.18 (SDIO_D0)
- new net SDC1_D1: J?.1 (Pin_1), U?.1, U?.19 (SDIO_D1)
- new net SDC1_D2: J?.6 (Pin_6), U?.1, U?.14 (SDIO_D2)
- new net SDC1_D3: J?.5 (Pin_5), U?.1, U?.15 (SDIO_D3)
- new net WL_H_WK: U?.13 (WL_H_WK)
