File: hardware/PCB/gpio.sch (KiCad schematic (older format))
At the start: 2 parts

Commit message: update pcb,
Parts:
- added R? (x4): R103,0603, Resistor_SMD:R_0603_1608Metric_Pad1.05x0.95mm_HandSolder, symbol taobao-r:R103,0603
- added SW? (x4): SW_Push, symbol Switch:SW_Push
Connections:
- net GND: now also R?.2, R?.2, R?.2, R?.2
- new net: R?.1, SW?.2 (x4)
- new net FEL: SW?.1
- new net USER_BTN1: SW?.1
- new net USER_BTN2: SW?.1
- new net USER_BTN3: SW?.1
Other:
- note added: "POWER HEALTHY"
- moved on the sheet: D?, R?

Commit message: update rtl8723 circuit,
Parts:
- SW1, SW2, SW3, SW4: renamed from SW?; footprint (none) -> footprint-lib:SW_SPST_PTS645
- gave numbers to parts that had none: 6
Changed lines of the file:
@@
 $EndComp
 $Comp
-L taobao-led:LED_GREEN,0805 D?
+L taobao-led:LED_GREEN,0805 D2
 U 1 1 5E87DFFD
 P 2250 3450
-F 0 "D?" V 2296 3382 50  0000 R CNN
+F 0 "D2" V 2296 3382 50  0000 R CNN
 F 1 "LED_GREEN,0805" V 2205 3382 50  0000 R CNN
 F 2 "footprint-lib:LED_0805_2012Metric" V 2250 3450 50  0001 C CNN
@@
 $EndComp
 $Comp
-L taobao-r:R103,0805 R?
+L taobao-r:R103,0805 R2
 U 1 1 5E87E8BC
 P 2250 3850
-F 0 "R?" H 2309 3896 50  0000 L CNN
+F 0 "R2" H 2309 3896 50  0000 L CNN
 F 1 "R103,0805" H 2309 3805 50  0000 L CNN
 F 2 "Resistor_SMD:R_0805_2012Metric_Pad1.15x1.40mm_HandSolder" H 2250 3850 50  0001 C CNN
@@
 POWER HEALTHY
 $Comp
-L Switch:SW_Push SW?
+L Switch:SW_Push SW1
 U 1 1 5E8FDE4B
 P 4650 3300
-F 0 "SW?" V 4604 3448 50  0000 L CNN
+F 0 "SW1" V 4604 3448 50  0000 L CNN
 F 1 "SW_Push" V 4695 3448 50  0000 L CNN
-F 2 "" H 4650 3500 50  0001 C CNN
+F 2 "footprint-lib:SW_SPST_PTS645" H 4650 3500 50  0001 C CNN
 F 3 "~" H 4650 3500 50  0001 C CNN
 	1    4650 3300
@@
 $EndComp
 $Comp
-L taobao-r:R103,0603 R?
+L taobao-r:R103,0603 R3
 U 1 1 5E8FEAE0
 P 4650 3800
-F 0 "R?" H 4709 3846 50  0000 L CNN
+F 0 "R3" H 4709 3846 50  0000 L CNN
 F 1 "R103,0603" H 4709 3755 50  0000 L CNN
 F 2 "Resistor_SMD:R_0603_1608Metric_Pad1.05x0.95mm_HandSolder" H 4650 3800 50  0001 C CNN
@@
 	4650 2650 4650 3100
 $Comp
-L Switch:SW_Push SW?
+L Switch:SW_Push SW2
 U 1 1 5E901C21
 P 6500 3300
-F 0 "SW?" V 6454 3448 50  0000 L CNN
+F 0 "SW2" V 6454 3448 50  0000 L CNN
 F 1 "SW_Push" V 6545 3448 50  0000 L CNN
-F 2 "" H 6500 3500 50  0001 C CNN
+F 2 "footprint-lib:SW_SPST_PTS645" H 6500 3500 50  0001 C CNN
 F 3 "~" H 6500 3500 50  0001 C CNN
 	1    6500 3300
@@
 $EndComp
 $Comp
-L taobao-r:R103,0603 R?
+L taobao-r:R103,0603 R4
 U 1 1 5E901C2B
 P 6500 3800
-F 0 "R?" H 6559 3846 50  0000 L CNN
+F 0 "R4" H 6559 3846 50  0000 L CNN
 F 1 "R103,0603" H 6559 3755 50  0000 L CNN
 F 2 "Resistor_SMD:R_0603_1608Metric_Pad1.05x0.95mm_HandSolder" H 6500 3800 50  0001 C CNN
@@
 	6500 2650 6500 3100
 $Comp
-L Switch:SW_Push SW?
+L Switch:SW_Push SW3
 U 1 1 5E906663
 P 7100 3300
-F 0 "SW?" V 7054 3448 50  0000 L CNN
+F 0 "SW3" V 7054 3448 50  0000 L CNN
 F 1 "SW_Push" V 7145 3448 50  0000 L CNN
-F 2 "" H 7100 3500 50  0001 C CNN
+F 2 "footprint-lib:SW_SPST_PTS645" H 7100 3500 50  0001 C CNN
 F 3 "~" H 7100 3500 50  0001 C CNN
 	1    7100 3300
@@
 $EndComp
 $Comp
-L taobao-r:R103,0603 R?
+L taobao-r:R103,0603 R5
 U 1 1 5E90666D
 P 7100 3800
-F 0 "R?" H 7159 3846 50  0000 L CNN
+F 0 "R5" H 7159 3846 50  0000 L CNN
 F 1 "R103,0603" H 7159 3755 50  0000 L CNN
 F 2 "Resistor_SMD:R_0603_1608Metric_Pad1.05x0.95mm_HandSolder" H 7100 3800 50  0001 C CNN
@@
 	7100 2650 7100 3100
 $Comp
-L Switch:SW_Push SW?
+L Switch:SW_Push SW4
 U 1 1 5E907E71
 P 7700 3300
-F 0 "SW?" V 7654 3448 50  0000 L CNN
+F 0 "SW4" V 7654 3448 50  0000 L CNN
 F 1 "SW_Push" V 7745 3448 50  0000 L CNN
-F 2 "" H 7700 3500 50  0001 C CNN
+F 2 "footprint-lib:SW_SPST_PTS645" H 7700 3500 50  0001 C CNN
 F 3 "~" H 7700 3500 50  0001 C CNN
 	1    7700 3300
@@
 $EndComp
 $Comp
-L taobao-r:R103,0603 R?
+L taobao-r:R103,0603 R6
 U 1 1 5E907E7B
 P 7700 3800
-F 0 "R?" H 7759 3846 50  0000 L CNN
+F 0 "R6" H 7759 3846 50  0000 L CNN
 F 1 "R103,0603" H 7759 3755 50  0000 L CNN
 F 2 "Resistor_SMD:R_0603_1608Metric_Pad1.05x0.95mm_HandSolder" H 7700 3800 50  0001 C CNN

Commit message: update,
Parts:
- SW1: value SW_Push -> FEL
Changed lines of the file:
@@
 $Descr A4 11693 8268
 encoding utf-8
-Sheet 4 6
+Sheet 3 6
 Title ""
 Date ""
@@
 $EndDescr
 $Comp
-L customized_power:+5V #PWR0125
+L customized_power:+5V #PWR011
 U 1 1 5E87D304
 P 2250 3000
-F 0 "#PWR0125" H 2250 2850 50  0001 C CNN
+F 0 "#PWR011" H 2250 2850 50  0001 C CNN
 F 1 "+5V" H 2265 3173 50  0000 C CNN
 F 2 "" H 2250 3000 50  0001 C CNN
@@
 $EndComp
 $Comp
-L power:GND #PWR0126
+L power:GND #PWR012
 U 1 1 5E87D54D
 P 2250 4050
-F 0 "#PWR0126" H 2250 3800 50  0001 C CNN
+F 0 "#PWR012" H 2250 3800 50  0001 C CNN
 F 1 "GND" H 2255 3877 50  0000 C CNN
 F 2 "" H 2250 4050 50  0001 C CNN
@@
 P 4650 3300
 F 0 "SW1" V 4604 3448 50  0000 L CNN
-F 1 "SW_Push" V 4695 3448 50  0000 L CNN
+F 1 "FEL" V 4695 3448 50  0000 L CNN
 F 2 "footprint-lib:SW_SPST_PTS645" H 4650 3500 50  0001 C CNN
 F 3 "~" H 4650 3500 50  0001 C CNN
@@
 	4650 3500 4650 3700
 $Comp
-L power:GND #PWR0127
+L power:GND #PWR013
 U 1 1 5E8FF449
 P 4650 4100
-F 0 "#PWR0127" H 4650 3850 50  0001 C CNN
+F 0 "#PWR013" H 4650 3850 50  0001 C CNN
 F 1 "GND" H 4655 3927 50  0000 C CNN
 F 2 "" H 4650 4100 50  0001 C CNN
@@
 	6500 3500 6500 3700
 $Comp
-L power:GND #PWR0128
+L power:GND #PWR014
 U 1 1 5E901C36
 P 6500 4100
-F 0 "#PWR0128" H 6500 3850 50  0001 C CNN
+F 0 "#PWR014" H 6500 3850 50  0001 C CNN
 F 1 "GND" H 6505 3927 50  0000 C CNN
 F 2 "" H 6500 4100 50  0001 C CNN
@@
 	7100 3500 7100 3700
 $Comp
-L power:GND #PWR0129
+L power:GND #PWR015
 U 1 1 5E906678
 P 7100 4100
-F 0 "#PWR0129" H 7100 3850 50  0001 C CNN
+F 0 "#PWR015" H 7100 3850 50  0001 C CNN
 F 1 "GND" H 7105 3927 50  0000 C CNN
 F 2 "" H 7100 4100 50  0001 C CNN
@@
 	7700 3500 7700 3700
 $Comp
-L power:GND #PWR0130
+L power:GND #PWR016
 U 1 1 5E907E86
 P 7700 4100
-F 0 "#PWR0130" H 7700 3850 50  0001 C CNN
+F 0 "#PWR016" H 7700 3850 50  0001 C CNN
 F 1 "GND" H 7705 3927 50  0000 C CNN
 F 2 "" H 7700 4100 50  0001 C CNN
